File: bluetooth_version.sch (EAGLE design)
At the start: 5 parts

Commit message: Bluetooth version check-in
Parts:
- removed SW1: (no value), Adafruit nRF52 Bluefruit Feather rev G:MICROBUILDER_SWITCH_TACT_SMT4.6X2.8
- removed U2: (no value), Adafruit nRF52 Bluefruit Feather rev G:MICROBUILDER_VREG_SOT23-5
- removed X1: (no value), Adafruit nRF52 Bluefruit Feather rev G:MICROBUILDER_CON_JST_PH_2PIN
- removed X2: (no value), Adafruit nRF52 Bluefruit Feather rev G:MICROBUILDER_JTAG-CORTEXBOXPOSTS
- added BT1: BK-912, BK-912:BK-912
- added C1: 10nF, SparkFun-Capacitors:10NF-0603-50V-10%
- added C2: 0.1uF, SparkFun-Capacitors:0.1UF-0603-25V-(+80/-20%)
- added C3: 15pF, SparkFun-Capacitors:15PF-0603-50V-5%
- added D1: BLUE, SparkFun-LED:LED-BLUE0603
- added IC1: BLUENRG-M2SP, SamacSys_Parts:BLUENRG-M2SP
- added J1: (no value), SparkFun-Connectors:CONN_05
- added J2: 455-1750-1-ND, SparkFun-Connectors:CONN_03
- added R1: 10k, SparkFun-Resistors:10KOHM-0603-1/10W-1%
- added R2: 820, SparkFun-Resistors:8.2KOHM-0603-1/10W-5%
- added R3: 47k, SparkFun-Resistors:47KOHM-0603-1/10W-1%
- added R4, R5, R6: 4.7k, SparkFun-Resistors:4.7KOHM-0603-1/10W-1%
- added S1: MOMENTARY-SWITCH-SPST-SMD-4.6X2.8MM, SparkFun-Switches:MOMENTARY-SWITCH-SPST-SMD-4.6X2.8MM
- added S2: (no value), SparkFun-Switches:SWITCH-SPDT-SMD-RIGHT-ANGLE
- U1: value (none) -> MAX30205MTA+T21-0137I_T833-2_MXM-M; device Adafruit nRF52 Bluefruit Feather rev G:MICROBUILDER_NRF52832_MODULE_MDBT42 -> MAX30205:MAX30205MTA+T21-0137I_T833-2_MXM-M
Connections:
- removed net 3.3V: X2.VCC
- removed net DFU: SW1.S, SW1.S1, U1.P0.20
- removed net SWO: X2.SWO
- new net BOOT: C3.1, IC1.DIO7/BOOT, R1.2, S1.1
- new net N$1: D1.A, R2.2
- new net N$2: BT1.+, S2.P
- new net OS: IC1.DIO0, R6.1, U1.OS
- new net RST: C1.1, IC1.RESETN, J1.5, R3.1
- new net RX: IC1.DIO11, J2.2
- new net TEST: IC1.ANATEST0/DIO14, R2.1
- new net TX: IC1.DIO8, J2.1
- new net VIN: C2.1, IC1.VIN, J1.1, R3.2, R4.2, R5.2, R6.2, S1.2, S2.S, U1.VDD
- net GND: now also BT1.-, C1.2, C2.2, C3.2, D1.C, IC1.GND, J1.3, J2.3, R1.1, U1.A0, U1.A1, U1.A2, U1.EPAD, U1.GND; no longer SW1.P, SW1.P1, U1.GND@1, U1.GND@4, X2.GND@1, X2.GND@2, X2.GNDDETECT, X2.KEY
- net SCL: now also IC1.DIO4, R5.1, U1.SCL; no longer U1.P0.26
- net SDA: now also IC1.DIO5, R4.1, U1.SDA; no longer U1.P0.25
- net SWCLK: now also IC1.DIO9, J1.2; no longer X2.SWDCLK
- net SWDIO: now also IC1.DIO10, J1.4; no longer X2.SWDIO
